File: keyboard.kicad_pcb (KiCad board)
At the start: 2 copper layers, 157 parts, among them J1 USB_C_Receptacle, SW1 SW_Push, U1 ATmega32U4-AU, Y1 16MHz

Commit message: Changed PCB layout
Parts:
- D68, D69, R5, R6: moved to B.Cu
- R1: moved to F.Cu
- moved R1 41.2 mm to (360.3, 112.2), turned to 225 degrees
- moved D67 33.9 mm to (328.7, 93.1)
- moved R8 33.9 mm to (322.3, 93.1)
- moved F1 31.8 mm to (355.0, 105.5), turned to 90 degrees
- moved C4 27.7 mm to (376.5, 117.0), turned to 135 degrees
- moved C6 27.7 mm to (367.5, 108.8), turned to 45 degrees
- moved C3 27.5 mm to (371.8, 120.2), turned to 315 degrees
- moved C7 25.6 mm to (345.3, 104.2), turned to 135 degrees
- moved C2 24.2 mm to (368.4, 115.5), turned to 225 degrees
- moved C1 23.9 mm to (343.7, 123.1), turned to 315 degrees
- moved R7 23.7 mm to (344.4, 105.3), turned to 90 degrees
- moved C5 23.5 mm to (372.1, 111.9), turned to 315 degrees
- moved Y1 23.2 mm to (342.0, 107.5), turned to 225 degrees
- moved D69 17.8 mm to (370.2, 100.8), turned to 270 degrees
- moved R4 17.5 mm to (343.7, 128.1), turned to 270 degrees
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Other:
- net class Default: trace_width 0.25 -> 0.254
- net class Power added: clearance 0.2, trace_width 0.381, via_dia 0.8, via_drill 0.4

Commit message: Finished routing, filled in ground planes, checked with DRC and 3D render
Parts:
- added M2_2.2mm: MountingHole_2.2mm_M2, MountingHole:MountingHole_2.2mm_M2, F.Cu at (149.4, 159.6)
- added M2_2.2mm: MountingHole_2.2mm_M2, MountingHole:MountingHole_2.2mm_M2, F.Cu at (288.3, 121.4)
- added M2_2.2mm: MountingHole_2.2mm_M2, MountingHole:MountingHole_2.2mm_M2, F.Cu at (65.5, 139.7)
- added M2_2.2mm: MountingHole_2.2mm_M2, MountingHole:MountingHole_2.2mm_M2, F.Cu at (357.2, 100.8)
- added M2_2.2mm: MountingHole_2.2mm_M2, MountingHole:MountingHole_2.2mm_M2, F.Cu at (357.2, 200.8)
- added M2_2.2mm: MountingHole_2.2mm_M2, MountingHole:MountingHole_2.2mm_M2, F.Cu at (36.5, 100.8)
- added M2_2.2mm: MountingHole_2.2mm_M2, MountingHole:MountingHole_2.2mm_M2, F.Cu at (36.5, 200.8)
- added REF**: MountingHole_2.2mm_M2, MountingHole:MountingHole_2.2mm_M2, F.Cu at (220.6, 140.8)
- added REF**: MountingHole_2.2mm_M2, MountingHole:MountingHole_2.2mm_M2, F.Cu at (202.6, 192.9)
- R1: moved to B.Cu
- moved R8 38.0 mm to (357.5, 107.4), turned to 270 degrees
- moved D69 34.0 mm to (336.7, 106.6)
- moved C3 33.0 mm to (339.0, 122.8), turned to 90 degrees
- moved D68 32.0 mm to (340.0, 106.6)
- moved C4 30.5 mm to (346.6, 122.9), turned to 0 degrees
- moved C2 29.5 mm to (339.0, 118.0), turned to 270 degrees
- moved R1 28.7 mm to (336.6, 128.3), turned to 0 degrees
- moved D67 28.0 mm to (352.8, 107.4), turned to 270 degrees
- moved C5 26.3 mm to (346.6, 118.4), turned to 0 degrees
- moved C6 26.2 mm to (342.2, 115.6), turned to 180 degrees
- moved C7 22.3 mm to (355.0, 124.2), turned to 0 degrees
- moved Y1 17.7 mm to (355.0, 119.5), turned to 90 degrees
- moved C8 16.8 mm to (354.9, 114.9), turned to 180 degrees
- moved C1 16.5 mm to (343.3, 106.6), turned to 90 degrees
- moved R4 11.1 mm to (353.6, 133.1), turned to 180 degrees
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Connections:
- U1 pad 1: Net-(U1-Pad1) -> COL2
- U1 pad 10: COL2 -> Net-(U1-Pad10)
- U1 pad 11: COL3 -> Net-(U1-Pad11)
- U1 pad 12: COL7 -> Net-(U1-Pad12)
- U1 pad 18: ROW0 -> Net-(U1-Pad18)
- U1 pad 19: ROW1 -> Net-(U1-Pad19)
- U1 pad 20: ROW2 -> ROW4
- U1 pad 22: ROW4 -> ROW2
- U1 pad 25: Net-(U1-Pad25) -> COL14
- U1 pad 26: Net-(U1-Pad26) -> COL13
- U1 pad 27: Net-(U1-Pad27) -> COL12
- U1 pad 28: COL4 -> COL11
- U1 pad 29: COL5 -> COL10
- U1 pad 30: COL6 -> COL9
- U1 pad 32: COL9 -> COL7
- U1 pad 36: Net-(U1-Pad36) -> ROW1
- U1 pad 37: COL14 -> ROW0
- U1 pad 38: COL13 -> COL6
- U1 pad 39: COL12 -> COL5
- U1 pad 40: COL11 -> COL4
- U1 pad 41: COL10 -> COL3
- U1 pad 8: COL0 -> COL1
- U1 pad 9: COL1 -> COL0
Routing:
- net COL0: track 0.00 -> 426.8 mm, vias 0 -> 1
- net COL1: track 0.00 -> 409.4 mm, vias 0 -> 1
- net COL2: track 0.00 -> 382.9 mm, vias 0 -> 1
- net ROW4: track 0.00 -> 363.3 mm
- net COL3: track 0.00 -> 339.5 mm, vias 0 -> 1
- net ROW3: track 0.00 -> 325.7 mm
- net COL5: track 0.00 -> 320.6 mm, vias 0 -> 1
- net COL4: track 0.00 -> 320.1 mm, vias 0 -> 1
- net ROW2: track 0.00 -> 314.1 mm
- net ROW0: track 0.00 -> 284.9 mm
- net COL6: track 0.00 -> 281.0 mm, vias 0 -> 1
- net ROW1: track 0.00 -> 276.0 mm
- net COL7: track 0.00 -> 273.8 mm, vias 0 -> 1
- net COL9: track 0.00 -> 260.7 mm, vias 0 -> 1
- net COL8: track 0.00 -> 256.3 mm, vias 0 -> 1
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- added copper zone on B.Cu, net GND
- added copper zone on F.Cu, net GND
Other:
- board outline added: 330.2 x 111.1 mm

Commit message: adjusted mounting holes, added dimension lines
Parts:
- removed the M2_2.2mm at (149.4, 159.6)
- removed the M2_2.2mm at (65.5, 139.7)
- removed REF** (x2): MountingHole_2.2mm_M2, MountingHole:MountingHole_2.2mm_M2
- added M2_2.2mm: MountingHole_2.2mm_M2, MountingHole:MountingHole_2.2mm_M2, F.Cu at (149.2, 159.5)
- added M2_2.2mm: MountingHole_2.2mm_M2, MountingHole:MountingHole_2.2mm_M2, F.Cu at (220.7, 140.5)
- added M2_2.2mm: MountingHole_2.2mm_M2, MountingHole:MountingHole_2.2mm_M2, F.Cu at (65.9, 139.7)
- added M2_2.2mm: MountingHole_2.2mm_M2, MountingHole:MountingHole_2.2mm_M2, F.Cu at (203.2, 192.9)
- moved M2_2.2mm 0.64 mm to (288.9, 121.4)
